Commit message: feat: update drok_gazebo sources

File: urdf/drok_gazebo.urdf (robot description, URDF)
Before this commit: robot DROK_CK, 9 links, 8 joints
Links:
- link BL: geometry collision cylinder length=0.035 radius=0.105; visual mesh filename=file:///home/ams7725/yunjae/Gazebo/DROK_CK/src/drok_gazebo/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
- link BLF: geometry collision box size=0.35 0.035 0.12; visual mesh filename=file:///home/ams7725/yunjae/Gazebo/DROK_CK/src/drok_gazebo/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
- link BR: geometry collision cylinder length=0.035 radius=0.105; visual mesh filename=file:///home/ams7725/yunjae/Gazebo/DROK_CK/src/drok_gazebo/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
- link BRF: geometry collision box size=0.35 0.035 0.12; visual mesh filename=file:///home/ams7725/yunjae/Gazebo/DROK_CK/src/drok_gazebo/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
- link FL: geometry collision cylinder length=0.035 radius=0.105; visual mesh filename=file:///home/ams7725/yunjae/Gazebo/DROK_CK/src/drok_gazebo/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
- link FLF: geometry collision box size=0.35 0.035 0.12; visual mesh filename=file:///home/ams7725/yunjae/Gazebo/DROK_CK/src/drok_gazebo/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
- link FR: geometry collision cylinder length=0.035 radius=0.105; visual mesh filename=file:///home/ams7725/yunjae/Gazebo/DROK_CK/src/drok_gazebo/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
- link FRF: geometry collision box size=0.35 0.035 0.12; visual mesh filename=file:///home/ams7725/yunjae/Gazebo/DROK_CK/src/drok_gazebo/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
Joints:
- joint BLF_joint: limit lower=0 upper=0 effort=30.0 velocity=2.0 -> lower=-1.57 upper=1.57 effort=30.0 velocity=2.0
- joint BL_JOINT: limit effort=3000.0 velocity=100.0 -> (none)
- joint BRF_joint: limit lower=0 upper=0 effort=30.0 velocity=2.0 -> lower=-1.57 upper=1.57 effort=30.0 velocity=2.0
- joint BR_JOINT: limit effort=3000.0 velocity=100.0 -> (none)
- joint FLF_joint: limit lower=0 upper=0 effort=30.0 velocity=2.0 -> lower=-1.57 upper=1.57 effort=30.0 velocity=2.0
- joint FL_JOINT: limit effort=3000.0 velocity=100.0 -> (none)
- joint FRF_joint: limit lower=0 upper=0 effort=30.0 velocity=2.0 -> lower=-1.57 upper=1.57 effort=30.0 velocity=2.0
- joint FR_JOINT: limit effort=3000.0 velocity=100.0 -> (none)

Commit message: Update configuration files and URDF

File: urdf/drok_gazebo.urdf (robot description, URDF)
Before this commit: robot DROK_CK, 9 links, 8 joints
Links:
- added link left_track, mass 1.0; collision box size=0.45 0.05 0.04; collision cylinder length=0.05 radius=0.105
- added link right_track, mass 1.0; collision box size=0.45 0.05 0.04; collision cylinder length=0.05 radius=0.105
- link BL: geometry visual mesh filename=file:///home/ams7725/yunjae/Gazebo/DROK_CK/src/drok_gazebo/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
- link BR: geometry visual mesh filename=file:///home/ams7725/yunjae/Gazebo/DROK_CK/src/drok_gazebo/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
- link FL: geometry visual mesh filename=file:///home/ams7725/yunjae/Gazebo/DROK_CK/src/drok_gazebo/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
- link FR: geometry visual mesh filename=file:///home/ams7725/yunjae/Gazebo/DROK_CK/src/drok_gazebo/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
Joints:
- added joint left_track_joint: type fixed, parent base_link, child left_track, origin xyz=0 0.1836 0 rpy=0 0 0
- added joint right_track_joint: type fixed, parent base_link, child right_track, origin xyz=0 -0.1836 0 rpy=0 0 0
